File: ART/board.sch (EAGLE design)
At the start: 10 parts, among them J1 455-1750-1-ND, J2 455-1750-1-ND, J3 455-1750-1-ND, U1 328P, Y1 16MHz

Commit message: fixed #3
Parts:
- added R1: 10k, adafruit:R-US_0207/9
Connections:
- net RESET: now also R1.2
- net VCC: now also R1.1
Changed lines of the file:
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@@
 <part name="J2" library="SparkFun-Connectors" deviceset="CONN_03" device="" value="455-1750-1-ND"/>
 <part name="J3" library="SparkFun-Connectors" deviceset="CONN_03" device="" value="455-1750-1-ND"/>
+<part name="R1" library="adafruit" library_urn="urn:adsk.eagle:library:420" deviceset="R-US_" device="0207/9" package3d_urn="urn:adsk.eagle:package:6240935/1" value="10k"/>
+<part name="P+3" library="supply1" library_urn="urn:adsk.eagle:library:371" deviceset="VCC" device=""/>
 </parts>
 <sheets>
@@
 <attribute name="VALUE" x="86.36" y="75.946" size="1.778" layer="96" font="vector" rot="R180"/>
 <attribute name="NAME" x="86.36" y="62.992" size="1.778" layer="95" font="vector" rot="R180"/>
+</instance>
+<instance part="R1" gate="G$1" x="-5.08" y="76.2" smashed="yes">
+<attribute name="NAME" x="-8.89" y="77.6986" size="1.778" layer="95"/>
+<attribute name="VALUE" x="-8.89" y="72.898" size="1.778" layer="96"/>
+</instance>
+<instance part="P+3" gate="VCC" x="-17.78" y="76.2" smashed="yes" rot="R90">
+<attribute name="VALUE" x="-15.24" y="73.66" size="1.778" layer="96" rot="R180"/>
 </instance>
 </instances>
@@
 <label x="71.12" y="71.12" size="1.778" layer="95"/>
 </segment>
+<segment>
+<pinref part="P+3" gate="VCC" pin="VCC"/>
+<pinref part="R1" gate="G$1" pin="1"/>
+<wire x1="-15.24" y1="76.2" x2="-10.16" y2="76.2" width="0.1524" layer="91"/>
+</segment>
 </net>
 <net name="RESET" class="0">
@@
 <junction x="12.7" y="76.2"/>
 <label x="2.54" y="76.2" size="1.778" layer="95"/>
+<pinref part="R1" gate="G$1" pin="2"/>
+<wire x1="12.7" y1="76.2" x2="0" y2="76.2" width="0.1524" layer="91"/>
 </segment>
 <segment>
